File: 02_Elements/H4_MainController_Rev_1/02_HW/H4_MainController_Rev_1.sch (EAGLE design)
At the start: 68 parts

Commit message: Finished H4_MainController_Rev_1
Finished design and Gerber Files of H4_MainController_Rev_1.

I sometimes wonder if this will be ever read even by a machine.
Parts:
- removed J_CON_04, J_CON_05, J_LED_00, J_LED_01: (no value), SparkFun-Connectors:M022.54MM_SCREWTERM
Connections:
- removed net GND1: J_CON_05.1
- removed net I2C_SCL1: J_CON_05.2
- removed net I2C_SDA1: J_CON_04.1
- net 5V: no longer J_LED_00.2
- net GND: no longer J_LED_01.2
- net LED_OUT: no longer J_LED_00.1
- net VIN: no longer J_CON_00.2, J_CON_02.2
- net VIN1: now also J_CON_00.2, J_CON_02.2; no longer J_CON_04.2
Other:
- moved on the sheet: J_CON_02, J_CON_03
