File: 02_Elements/H4_MainController_Rev_1/02_HW/H4_MainController_Rev_1.brd (EAGLE design)
At the start: 70 x 17 mm, 68 parts

Commit message: Finished H4_MainController_Rev_1
Finished design and Gerber Files of H4_MainController_Rev_1.

I sometimes wonder if this will be ever read even by a machine.
Parts:
- removed J_CON_04, J_CON_05, J_LED_00, J_LED_01: (no value), SparkFun-Connectors:1X02_2.54_SCREWTERM
- moved J_PWSW 350.8 mm to (84.2, 64.0), turned to 180 degrees
- moved J_PWSW_0 345.3 mm to (79.2, 64.0), turned to 180 degrees
- moved R_MIDI_0 324.4 mm to (80.0, 42.5)
- moved R_MIDI_1 310.7 mm to (80.0, 32.5)
- moved J_PW 306.5 mm to (89.0, 54.0), turned to 90 degrees
- moved J_MIDI 305.9 mm to (91.0, 37.0), turned to 90 degrees
- moved J_SW_03 284.1 mm to (51.2, 64.0), turned to 180 degrees
- moved J_SW_02 280.1 mm to (56.2, 64.0), turned to 180 degrees
- moved R_SW_RST 278.4 mm to (89.5, 63.5), turned to 270 degrees
- moved J_SW_01 278.1 mm to (65.0, 64.0), turned to 180 degrees
- moved J_SW_00 274.6 mm to (70.0, 64.0), turned to 180 degrees
- moved SW_RST 274.4 mm to (95.0, 64.0)
- moved R_SW_02 245.5 mm to (38.0, 11.0), turned to 180 degrees
- moved SW_02 232.1 mm to (38.0, 5.00), turned to 270 degrees
- moved C_LED_ARD_00 207.8 mm to (64.0, 15.0), turned to 90 degrees
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Connections:
- removed net GND1: J_CON_05.P1
- removed net I2C_SCL1: J_CON_05.P2
- removed net I2C_SDA1: J_CON_04.P1
- net 5V: no longer J_LED_00.P2
- net GND: no longer J_LED_01.P2
- net LED_OUT: no longer J_LED_00.P1
- net VIN: no longer J_CON_00.P2, J_CON_02.P2
- net VIN1: now also J_CON_00.P2, J_CON_02.P2; no longer J_CON_04.P2
Routing:
- net GND: track 103.6 -> 383.3 mm, vias 7 -> 5
- net 5V: track 104.2 -> 376.6 mm
- net SW_02: track 0.00 -> 135.4 mm, vias 0 -> 1
- net SW_RST: track 0.00 -> 105.9 mm, vias 0 -> 1
- net SW_00: track 0.00 -> 102.8 mm
- net SW_01: track 0.00 -> 71.1 mm
- net N$7: track 0.00 -> 58.9 mm, vias 0 -> 2
- net N$11: track 0.00 -> 58.8 mm, vias 0 -> 2
- net N$2: track 0.00 -> 56.5 mm, vias 0 -> 2
- net VIN: track 75.0 -> 131.3 mm
- net N$1: track 0.00 -> 56.3 mm, vias 0 -> 1
- net N$8: track 0.00 -> 46.3 mm, vias 0 -> 2
- net TX: track 0.00 -> 33.3 mm
- net N$16: track 0.00 -> 29.1 mm
- net N$6: track 0.00 -> 28.5 mm
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- added copper zone on layer 1, net N$18
- added copper zone on layer 16, net N$19
- removed copper zone on layer 16, net FILLBOT
- removed copper zone on layer 1, net FILLTOP
Other:
- board size 70 x 17 mm -> 100 x 75 mm
- board text added: "3V3 GND D15 D2 D4 RX2 TX2 D5 D18 D19 D21 RX0 TX0 D22 D23"
- board text added: "Autofabricantes Un instrumento para Henar Spain, 2022"
- board text added: "C:/Users/PablodMM/Google Drive/Henar #3/03_Recursos/License_3_0_Logo.bmp"
- board text added: "C_LED_00"
- board text added: "C_LED_01"
- board text added: "C_LED_02"
- board text added: "C_LED_03"
- board text added: "C_LED_04"
- board text added: "C_LED_05"
- board text added: "C_LED_ARD_00"
- board text added: "C_LED_ARD_01"
- board text added: "H4_MainController_Rev_1"
- board text added: "INPUT POWER 7-12V"
- board text added: "J_MIDI"
- board text added: "J_PW"
- board text added: "J_PWSW_0/1"
- board text added: "J_SW_00/01"
- board text added: "J_SW_02/03"
- board text added: "L_RGB_ARD_00"
- board text added: "L_RGB_ARD_01"
- board text added: "Pablodmm.isp@gmail.com @lupin.o"
- board text added: "RAW GND RST VCC A3 A2 A1 A0 15 14 16 10"
- board text added: "R_ESP_I2C_0"
- board text added: "R_ESP_I2C_1"
- board text added: "R_I2C"
- board text added: "R_I2C ESP"
- board text added: "R_SW_0"
- board text added: "R_SW_1"
- board text added: "SW_00"
- board text added: "SW_01"
- board text added: "SW_02"
- board text added: "SW_PW"
- board text added: "SW_RST"
- board text added: "TX0 RX1 GND GND D2 D3 D4 D5 D6 D7 D8 D9"
- board text added: "VIN GND D13 D12 D14 D27 D26 D25 D33 D32 D35 D34 VN VP EN"
- board text removed: "5V"
- board text removed: "Autofabricantes / Un instrumento para Henar Spain, 2020"
- board text removed: "C_ATM_2"
- board text removed: "C_VR_0"
- board text removed: "H4_PadController_Rev_1"
- board text removed: "I2C:"
- board text removed: "J_PROG"
- board text removed: "MISO"
- board text removed: "MOSI"
- board text removed: "RST"
- board text removed: "SCK"
- board text removed: "U_ATMEGA328"
- board text removed: "U_VR"
