File: 02_Elements/H4_PadController_Rev_2/01_Resources/H4_Pad_80x80mm.brd (EAGLE design)
At the start: 80 x 100 mm, 0 parts

Commit message: Wow I havent sleept today I'm on autopilot
Routing:
- net S$4: track 359.5 -> 353.5 mm
Other:
- outline, holes or cut-outs redrawn
Changed lines of the file:
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@@
 <layer number="14" name="Route14" color="1" fill="6" visible="no" active="no"/>
 <layer number="15" name="Route15" color="4" fill="6" visible="no" active="no"/>
-<layer number="16" name="Bottom" color="1" fill="1" visible="yes" active="yes"/>
+<layer number="16" name="Bottom" color="1" fill="1" visible="no" active="yes"/>
 <layer number="17" name="Pads" color="2" fill="1" visible="no" active="yes"/>
 <layer number="18" name="Vias" color="2" fill="1" visible="no" active="yes"/>
 <layer number="19" name="Unrouted" color="6" fill="1" visible="no" active="yes"/>
-<layer number="20" name="Dimension" color="15" fill="1" visible="yes" active="yes"/>
-<layer number="21" name="tPlace" color="7" fill="1" visible="yes" active="yes"/>
+<layer number="20" name="Dimension" color="15" fill="1" visible="no" active="yes"/>
+<layer number="21" name="tPlace" color="7" fill="1" visible="no" active="yes"/>
 <layer number="22" name="bPlace" color="7" fill="1" visible="no" active="yes"/>
 <layer number="23" name="tOrigins" color="15" fill="1" visible="no" active="yes"/>
@@
 <layer number="44" name="Drills" color="7" fill="1" visible="no" active="yes"/>
 <layer number="45" name="Holes" color="7" fill="1" visible="no" active="yes"/>
-<layer number="46" name="Milling" color="3" fill="1" visible="no" active="yes"/>
+<layer number="46" name="Milling" color="3" fill="1" visible="yes" active="yes"/>
 <layer number="47" name="Measures" color="7" fill="1" visible="no" active="yes"/>
 <layer number="48" name="Document" color="7" fill="1" visible="no" active="yes"/>
@@
 <board>
 <plain>
-<wire x1="4" y1="2" x2="2" y2="4" width="0" layer="19" curve="-90"/>
-<wire x1="2" y1="4" x2="2" y2="76" width="0" layer="19"/>
-<wire x1="2" y1="76" x2="4" y2="78" width="0" layer="19" curve="-90"/>
-<wire x1="4" y1="78" x2="76" y2="78" width="0" layer="19"/>
-<wire x1="76" y1="78" x2="78" y2="76" width="0" layer="19" curve="-90"/>
-<wire x1="78" y1="76" x2="78" y2="4" width="0" layer="19"/>
-<wire x1="78" y1="4" x2="76" y2="2" width="0" layer="19" curve="-90"/>
-<wire x1="76" y1="2" x2="4" y2="2" width="0" layer="19"/>
+<wire x1="6" y1="3" x2="3" y2="5" width="0" layer="46" curve="-90"/>
+<wire x1="3" y1="5" x2="3" y2="76" width="0" layer="46"/>
+<wire x1="3" y1="76" x2="5" y2="78" width="0" layer="46" curve="-90"/>
+<wire x1="5" y1="78" x2="75" y2="78" width="0" layer="46"/>
+<wire x1="75" y1="78" x2="77" y2="76" width="0" layer="46" curve="-90"/>
+<wire x1="77" y1="76" x2="77" y2="5" width="0" layer="46"/>
+<wire x1="77" y1="5" x2="75" y2="3" width="0" layer="46" curve="-90"/>
+<wire x1="75" y1="3" x2="6" y2="3" width="0" layer="46"/>
 <wire x1="0" y1="3" x2="0" y2="97" width="0" layer="21"/>
 <wire x1="0" y1="97" x2="3" y2="100" width="0" layer="21" curve="-90"/>
@@
 <wire x1="19" y1="84" x2="20" y2="83" width="0" layer="1" curve="-90"/>
 <wire x1="20" y1="83" x2="20" y2="75" width="0" layer="1"/>
-<wire x1="14" y1="75" x2="7" y2="75" width="0" layer="1"/>
-<wire x1="5" y1="73" x2="5" y2="7" width="0" layer="1"/>
-<wire x1="7" y1="5" x2="73" y2="5" width="0" layer="1"/>
-<wire x1="75" y1="7" x2="75" y2="73" width="0" layer="1"/>
+<wire x1="14" y1="75" x2="8" y2="75" width="0" layer="1"/>
+<wire x1="6" y1="73" x2="6" y2="8" width="0" layer="1"/>
+<wire x1="8" y1="6" x2="72" y2="6" width="0" layer="1"/>
+<wire x1="74" y1="8" x2="74" y2="73" width="0" layer="1"/>
 <wire x1="60" y1="83" x2="61" y2="84" width="0" layer="1" curve="-90"/>
 <wire x1="61" y1="84" x2="64" y2="84" width="0" layer="1"/>
@@
 <wire x1="65" y1="83" x2="65" y2="75" width="0" layer="1"/>
 <wire x1="60" y1="83" x2="60" y2="75" width="0" layer="1"/>
-<wire x1="73" y1="75" x2="65" y2="75" width="0" layer="1"/>
+<wire x1="72" y1="75" x2="65" y2="75" width="0" layer="1"/>
 <wire x1="51" y1="83" x2="52" y2="84" width="0" layer="1" curve="-90"/>
 <wire x1="52" y1="84" x2="55" y2="84" width="0" layer="1"/>
@@
 <wire x1="42" y1="75" x2="38" y2="75" width="0" layer="1"/>
 <wire x1="33" y1="75" x2="20" y2="75" width="0" layer="1"/>
-<wire x1="7" y1="5" x2="5" y2="7" width="0" layer="1" curve="-90"/>
-<wire x1="73" y1="5" x2="75" y2="7" width="0" layer="1" curve="90"/>
-<wire x1="75" y1="73" x2="73" y2="75" width="0" layer="1" curve="90"/>
-<wire x1="5" y1="73" x2="7" y2="75" width="0" layer="1" curve="-90"/>
+<wire x1="8" y1="6" x2="6" y2="8" width="0" layer="1" curve="-90"/>
+<wire x1="72" y1="6" x2="74" y2="8" width="0" layer="1" curve="90"/>
+<wire x1="74" y1="73" x2="72" y2="75" width="0" layer="1" curve="90"/>
+<wire x1="6" y1="73" x2="8" y2="75" width="0" layer="1" curve="-90"/>
 </signal>
 </signals>
